Commit message: Update robot.urdf

File: robot.urdf (robot description, URDF)
Before this commit: robot robot, 5 links, 4 joints
Links:
- added link lidar_link; collision cylinder length=0.06 radius=0.03; visual cylinder length=0.03 radius=0.03
- link caster_wheel: geometry collision sphere radius=0.015; visual sphere radius=0.015
- link chassis: geometry collision mesh filename=package://mobile-0244/stl/assbodynew.STL scale=0.001 0.001 0.001; visual mesh filename=package://mobile-0244/stl/assbodynew.STL scale=0.001 0.001 0.001
Joints:
- added joint lidar_joint: type fixed, parent chassis, child lidar_link, origin xyz=0 0 0.15 rpy=0 0 0
